Commit message: themis retarget

File: src/holosoma_retargeting/holosoma_retargeting/models/themis/themis_28dof.urdf (robot description, URDF)
Before this commit: robot TH02-A7, 29 links, 28 joints
Joints:
- joint ANKLE_PITCH_L: limit lower=-3.14 upper=3.14 effort=35 velocity=30 -> lower=-0.8 upper=0.8 effort=100 velocity=10
- joint ANKLE_PITCH_R: limit lower=-3.14 upper=3.14 effort=35 velocity=30 -> lower=-0.8 upper=0.8 effort=100 velocity=10
- joint ANKLE_ROLL_L: limit lower=-1.56 upper=1.56 effort=35 velocity=30 -> lower=-0.5 upper=0.5 effort=100 velocity=10
- joint ANKLE_ROLL_R: limit lower=-1.56 upper=1.56 effort=35 velocity=30 -> lower=-0.5 upper=0.5 effort=100 velocity=10
- joint HIP_PITCH_L: limit lower=-1.56 upper=1.56 effort=150 velocity=30 -> lower=-1.56 upper=1.56 effort=100 velocity=10
- joint HIP_PITCH_R: limit lower=-1.56 upper=1.56 effort=150 velocity=30 -> lower=-1.56 upper=1.56 effort=100 velocity=10
- joint HIP_ROLL_L: limit lower=-1.56 upper=1.56 effort=150 velocity=30 -> lower=-1.56 upper=1.56 effort=100 velocity=10
- joint HIP_ROLL_R: limit lower=-1.56 upper=1.56 effort=150 velocity=30 -> lower=-1.56 upper=1.56 effort=100 velocity=10
- joint KNEE_PITCH_L: limit lower=0 upper=3.14 effort=150 velocity=30 -> lower=0.0 upper=3.14 effort=100 velocity=10
- joint KNEE_PITCH_R: limit lower=0 upper=3.14 effort=150 velocity=30 -> lower=0.0 upper=3.14 effort=100 velocity=10

Commit message: themis_running

File: src/holosoma_retargeting/holosoma_retargeting/models/themis/themis_28dof.urdf (robot description, URDF)
Before this commit: robot TH02-A7, 29 links, 28 joints
Links:
- added link FOOT_L_heel_link, mass 0.0
- added link FOOT_L_toe_link, mass 0.0
- added link FOOT_R_heel_link, mass 0.0
- added link FOOT_R_toe_link, mass 0.0
Joints:
- added joint FOOT_L_heel_joint: type fixed, parent FOOT_L, child FOOT_L_heel_link, origin xyz=0 0 0 rpy=0 0 0
- added joint FOOT_L_toe_joint: type fixed, parent FOOT_L, child FOOT_L_toe_link, origin xyz=0.05 0 0.12 rpy=0 0 0
- added joint FOOT_R_heel_joint: type fixed, parent FOOT_R, child FOOT_R_heel_link, origin xyz=0 0 0 rpy=0 0 0
- added joint FOOT_R_toe_joint: type fixed, parent FOOT_R, child FOOT_R_toe_link, origin xyz=0.05 0 0.12 rpy=0 0 0
