Commit message: themis urdf nominal model update

File: src/holosoma_retargeting/holosoma_retargeting/models/themis/themis_28dof_nominal_collison.urdf (robot description, URDF)
Before this commit: robot themis-29dof, 38 links, 37 joints
Links:
- added link FOOT_L_contact_geom_1, mass 0; collision sphere radius=0.005; visual sphere radius=0.005
- added link FOOT_L_contact_geom_2, mass 0; collision sphere radius=0.005; visual sphere radius=0.005
- added link FOOT_L_contact_geom_3, mass 0; collision sphere radius=0.005; visual sphere radius=0.005
- added link FOOT_L_contact_geom_4, mass 0; collision sphere radius=0.005; visual sphere radius=0.005
- added link FOOT_L_contact_geom_5, mass 0; collision sphere radius=0.005; visual sphere radius=0.005
- added link FOOT_L_contact_geom_6, mass 0; collision sphere radius=0.005; visual sphere radius=0.005
- added link FOOT_R_contact_geom_1, mass 0; collision sphere radius=0.005; visual sphere radius=0.005
- added link FOOT_R_contact_geom_2, mass 0; collision sphere radius=0.005; visual sphere radius=0.005
- added link FOOT_R_contact_geom_3, mass 0; collision sphere radius=0.005; visual sphere radius=0.005
- added link FOOT_R_contact_geom_4, mass 0; collision sphere radius=0.005; visual sphere radius=0.005
- added link FOOT_R_contact_geom_5, mass 0; collision sphere radius=0.005; visual sphere radius=0.005
- added link FOOT_R_contact_geom_6, mass 0; collision sphere radius=0.005; visual sphere radius=0.005
- link BASE_LINK: geometry collision mesh filename=meshes/BASE_LINK.STL
- link FOOT_L: geometry collision mesh filename=meshes/FOOT_L_rot2.STL
- link FOOT_L_contact: geometry collision sphere radius=0.005; visual sphere radius=0.005
- link FOOT_R: geometry collision mesh filename=meshes/FOOT_R_rot2.STL
- link FOOT_R_contact: geometry collision sphere radius=0.005; visual sphere radius=0.005
- link LOWERWRIST_L_contact: geometry collision sphere radius=0.04; visual sphere radius=0.04
- link LOWERWRIST_R_contact: geometry collision sphere radius=0.04; visual sphere radius=0.04
- link TIBIA_L: geometry collision mesh filename=meshes/TIBIA_L_rot.STL
- link TIBIA_R: geometry collision mesh filename=meshes/TIBIA_R_rot.STL
- link UPPERARM_L: geometry collision mesh filename=meshes/UPPERARM_L_rot.STL
- link UPPERARM_R: geometry collision mesh filename=meshes/UPPERARM_R_rot.STL
Joints:
- added joint FOOT_L_contact_to_FOOT_L_contact_geom_1: type fixed, parent FOOT_L_contact, child FOOT_L_contact_geom_1, origin xyz=0 0 0 rpy=0 0 0
- added joint FOOT_L_contact_to_FOOT_L_contact_geom_2: type fixed, parent FOOT_L_contact, child FOOT_L_contact_geom_2, origin xyz=0 0 0 rpy=0 0 0
- added joint FOOT_L_contact_to_FOOT_L_contact_geom_3: type fixed, parent FOOT_L_contact, child FOOT_L_contact_geom_3, origin xyz=0 0 0 rpy=0 0 0
- added joint FOOT_L_contact_to_FOOT_L_contact_geom_4: type fixed, parent FOOT_L_contact, child FOOT_L_contact_geom_4, origin xyz=0 0 0 rpy=0 0 0
- added joint FOOT_L_contact_to_FOOT_L_contact_geom_5: type fixed, parent FOOT_L_contact, child FOOT_L_contact_geom_5, origin xyz=0 0 0 rpy=0 0 0
- added joint FOOT_L_contact_to_FOOT_L_contact_geom_6: type fixed, parent FOOT_L_contact, child FOOT_L_contact_geom_6, origin xyz=0 0 0 rpy=0 0 0
- added joint FOOT_R_contact_to_FOOT_R_contact_geom_1: type fixed, parent FOOT_R_contact, child FOOT_R_contact_geom_1, origin xyz=0 0 0 rpy=0 0 0
- added joint FOOT_R_contact_to_FOOT_R_contact_geom_2: type fixed, parent FOOT_R_contact, child FOOT_R_contact_geom_2, origin xyz=0 0 0 rpy=0 0 0
- added joint FOOT_R_contact_to_FOOT_R_contact_geom_3: type fixed, parent FOOT_R_contact, child FOOT_R_contact_geom_3, origin xyz=0 0 0 rpy=0 0 0
- added joint FOOT_R_contact_to_FOOT_R_contact_geom_4: type fixed, parent FOOT_R_contact, child FOOT_R_contact_geom_4, origin xyz=0 0 0 rpy=0 0 0
- added joint FOOT_R_contact_to_FOOT_R_contact_geom_5: type fixed, parent FOOT_R_contact, child FOOT_R_contact_geom_5, origin xyz=0 0 0 rpy=0 0 0
- added joint FOOT_R_contact_to_FOOT_R_contact_geom_6: type fixed, parent FOOT_R_contact, child FOOT_R_contact_geom_6, origin xyz=0 0 0 rpy=0 0 0
- joint root_joint: origin xyz=0 0 0 rpy=0 0 0 -> xyz=0 0 1.17 rpy=0 0 0
